File: Hardware/PCB/multiples/multiples.kicad_pcb (KiCad board)
At the start: 2 copper layers, 7 parts, among them J1 Synth_power_2x5

Commit message: PCB layout
Parts:
- added C5: 100nF, ao_tht:C_Disc_D3.0mm_W1.6mm_P2.50mm, B.Cu at (139.7, 53.3)
- added C6: 100nF, ao_tht:C_Disc_D3.0mm_W1.6mm_P2.50mm, B.Cu at (141.0, 33.1)
- added GRAF1: Holes, multiples:multiples_panel_holes, F.Cu at (125.0, 100.0)
- added GRAF2: AO logo, ao_tht:analogoutput, B.Cu at (124.8, 88.3)
- added GRAF3: CC0 logo, ao_tht:CC0_logo, B.Cu at (107.8, 8.26)
- added J10: AudioJack2, ao_tht:Jack_6.35mm_PJ_629HAN, F.Cu at (137.5, 150.0)
- added J11: AudioJack2, ao_tht:Jack_6.35mm_PJ_629HAN, F.Cu at (137.5, 175.0)
- added J2: Synth_power_2x5, ao_tht:Power_Header, B.Cu at (123.2, 30.5)
- added J3: AudioJack2, ao_tht:Jack_6.35mm_PJ_629HAN, F.Cu at (112.5, 100.0)
- added J4: AudioJack2, ao_tht:Jack_6.35mm_PJ_629HAN, F.Cu at (112.5, 125.0)
- added J5: AudioJack2, ao_tht:Jack_6.35mm_PJ_629HAN, F.Cu at (112.5, 150.0)
- added J6: AudioJack2, ao_tht:Jack_6.35mm_PJ_629HAN, F.Cu at (112.5, 175.0)
- added J7: AudioJack2_SwitchT, ao_tht:Jack_6.35mm_PJ_629HAN, F.Cu at (137.5, 75.0)
- added J8: AudioJack2, ao_tht:Jack_6.35mm_PJ_629HAN, F.Cu at (137.5, 100.0)
- added J9: AudioJack2, ao_tht:Jack_6.35mm_PJ_629HAN, F.Cu at (137.5, 125.0)
- added R1: 1M, ao_tht:R_Axial_DIN0207_L6.3mm_D2.5mm_P10.16mm_Horizontal, B.Cu at (114.3, 53.3)
- added R10: 1k, ao_tht:R_Axial_DIN0207_L6.3mm_D2.5mm_P10.16mm_Horizontal, B.Cu at (144.8, 25.4)
- added R2: 1k, ao_tht:R_Axial_DIN0207_L6.3mm_D2.5mm_P10.16mm_Horizontal, B.Cu at (119.4, 63.5)
- added R3: 1k, ao_tht:R_Axial_DIN0207_L6.3mm_D2.5mm_P10.16mm_Horizontal, B.Cu at (104.1, 63.5)
- added R4: 1k, ao_tht:R_Axial_DIN0207_L6.3mm_D2.5mm_P10.16mm_Horizontal, B.Cu at (104.1, 25.4)
- added R5: 1k, ao_tht:R_Axial_DIN0207_L6.3mm_D2.5mm_P10.16mm_Horizontal, B.Cu at (111.8, 35.6)
- added R6: 1M, ao_tht:R_Axial_DIN0207_L6.3mm_D2.5mm_P10.16mm_Horizontal, B.Cu at (134.6, 53.3)
- added R7: 1k, ao_tht:R_Axial_DIN0207_L6.3mm_D2.5mm_P10.16mm_Horizontal, B.Cu at (144.8, 63.5)
- added R8: 1k, ao_tht:R_Axial_DIN0207_L6.3mm_D2.5mm_P10.16mm_Horizontal, B.Cu at (129.5, 63.5)
- added R9: 1k, ao_tht:R_Axial_DIN0207_L6.3mm_D2.5mm_P10.16mm_Horizontal, B.Cu at (137.2, 35.6)
- added U1: TL074, ao_tht:DIP-14_W7.62mm_Socket_LongPads, B.Cu at (119.4, 48.3)
- added U2: TL074, ao_tht:DIP-14_W7.62mm_Socket_LongPads, B.Cu at (144.8, 48.3)
- C1, C2: footprint Capacitor_THT:CP_Radial_D5.0mm_P2.00mm -> ao_tht:CP_Radial_D6.3mm_P2.50mm; moved to B.Cu
- C3, C4: value 0.1uF -> 100nF; footprint Capacitor_THT:C_Disc_D3.0mm_W1.6mm_P2.50mm -> ao_tht:C_Disc_D3.0mm_W1.6mm_P2.50mm; moved to B.Cu
- D1, D2: footprint Diode_THT:D_DO-41_SOD81_P7.62mm_Horizontal -> ao_tht:D_DO-41_SOD81_P7.62mm_Horizontal; moved to B.Cu
- J1: value Synth_power_2x5 -> AudioJack2_SwitchT; footprint ao_tht:Power_Header -> ao_tht:Jack_6.35mm_PJ_629HAN
- moved C2 158.1 mm to (104.1, 17.8), turned to 270 degrees
- moved C4 143.2 mm to (108.0, 33.0), turned to 270 degrees
- moved D2 133.7 mm to (116.8, 19.1), turned to 180 degrees
- moved C3 131.3 mm to (109.2, 53.3), turned to 270 degrees
- moved C1 117.3 mm to (144.8, 20.3), turned to 90 degrees
- moved J1 114.6 mm to (112.5, 75.0), turned to 270 degrees
- moved D1 111.3 mm to (139.7, 19.1), turned to 180 degrees
Routing:
- net Net-(J11-PadT): track 0.00 -> 154.0 mm
- net Net-(J6-PadT): track 0.00 -> 141.0 mm
- net Net-(J5-PadT): track 0.00 -> 124.8 mm
- net Net-(J10-PadT): track 0.00 -> 115.5 mm
- net -12V: track 0.00 -> 78.9 mm
- net +12V: track 0.00 -> 78.5 mm
- net Net-(J4-PadT): track 0.00 -> 75.9 mm
- net Net-(J9-PadT): track 0.00 -> 75.3 mm
- net Net-(J1-PadT): track 0.00 -> 59.2 mm
- net Net-(J8-PadT): track 0.00 -> 51.0 mm
- net Net-(J3-PadT): track 0.00 -> 49.4 mm
- net Net-(J7-PadT): track 0.00 -> 38.6 mm
- net Net-(R9-Pad2): track 0.00 -> 18.4 mm
- net Net-(R5-Pad2): track 0.00 -> 18.4 mm
- net /-12_IN: track 0.00 -> 16.6 mm
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- added copper zone on B.Cu, net GND
- added copper zone on F.Cu, net GND
Other:
- board outline added: 50 x 200 mm
- board text added: "Buffered Multiples"
- board text added: "Rich Holmes / August 2021 CC0 1.0 https://github.com/holmesrichards/mults"

Commit message: Clean up libraries, Schottky footprint update
Parts:
- D1, D2: footprint ao_tht:D_DO-41_SOD81_P7.62mm_Horizontal -> ao_tht:D_DO-41_SOD81_P10.16mm_Horizontal
- moved D2 16.5 mm to (116.8, 35.6), turned to 90 degrees
- moved D1 9.92 mm to (132.1, 25.4), turned to 270 degrees
- moved C1 8.89 mm to (135.9, 20.3)
- moved C2 8.89 mm to (113.0, 17.8)
Routing:
- net /+12_IN: track 9.42 -> 20.4 mm
- net -12V: track 78.9 -> 88.9 mm
- net +12V: track 78.5 -> 88.4 mm
- net /-12_IN: track 16.6 -> 11.0 mm

Commit message: Better .gitignore
Parts:
- added TP1: -12V, ao_tht:TestPoint_THTPad_D1.5mm_Drill0.7mm, F.Cu at (148.6, 22.9)
- added TP2: +12V, ao_tht:TestPoint_THTPad_D1.5mm_Drill0.7mm, F.Cu at (148.6, 8.89)
- added TP3: GND, ao_tht:TestPoint_THTPad_1.5x1.5mm_Drill0.7mm, F.Cu at (148.6, 15.8)
- moved GRAF3 2.86 mm to (104.9, 8.26)
Routing:
- net -12V: track 88.9 -> 106.6 mm
- net +12V: track 88.4 -> 101.4 mm
Other:
- net class Default removed
- net class Power removed

Commit message: KiCad 7, libraries to folder
Parts:
- C1, C2: footprint ao_tht:CP_Radial_D6.3mm_P2.50mm -> AO_tht:CP_Radial_D6.3mm_P2.50mm
- C3, C4, C5, C6: footprint ao_tht:C_Disc_D3.0mm_W1.6mm_P2.50mm -> AO_tht:C_Disc_D3.0mm_W1.6mm_P2.50mm
- D1, D2: footprint ao_tht:D_DO-41_SOD81_P10.16mm_Horizontal -> AO_tht:D_DO-41_SOD81_P10.16mm_Horizontal
- GRAF2: footprint ao_tht:analogoutput -> AO_tht:analogoutput
- GRAF3: footprint ao_tht:CC0_logo -> AO_tht:CC0_logo
- J1, J10, J11, J3, J4, J5, J6, J7, J8, J9: footprint ao_tht:Jack_6.35mm_PJ_629HAN -> AO_tht:Jack_6.35mm_PJ_629HAN_slots
- J2: footprint ao_tht:Power_Header -> AO_tht:Power_Header
- R1, R10, R2, R3, R4, R5, R6, R7, R8, R9: footprint ao_tht:R_Axial_DIN0207_L6.3mm_D2.5mm_P10.16mm_Horizontal -> AO_tht:R_Axial_DIN0207_L6.3mm_D2.5mm_P10.16mm_Horizontal
- TP1, TP2: footprint ao_tht:TestPoint_THTPad_D1.5mm_Drill0.7mm -> AO_tht:TestPoint_THTPad_D1.5mm_Drill0.7mm
- TP3: footprint ao_tht:TestPoint_THTPad_1.5x1.5mm_Drill0.7mm -> AO_tht:TestPoint_THTPad_D1.5mm_Drill0.7mm
- U1, U2: footprint ao_tht:DIP-14_W7.62mm_Socket_LongPads -> AO_tht:DIP-14_W7.62mm_Socket_LongPads
- moved GRAF3 196.3 mm to (200.0, 180.0)
- moved R1 84.1 mm to (189.3, 91.3)
- moved C1 84.1 mm to (210.9, 58.3)
- moved C2 84.1 mm to (188.0, 55.8)
- moved C3 84.1 mm to (184.2, 91.3)
- moved C5 84.1 mm to (214.7, 91.3)
- moved C6 84.1 mm to (216.0, 71.1)
- moved D1 84.1 mm to (207.1, 63.4)
- moved D2 84.1 mm to (191.8, 73.6)
- moved GRAF1 84.1 mm to (200.0, 138.0)
- moved GRAF2 84.1 mm to (199.8, 126.3)
- moved J1 84.1 mm to (187.5, 113.0)
- moved J10 84.1 mm to (212.5, 188.0)
- moved J11 84.1 mm to (212.5, 213.0)
- moved J2 84.1 mm to (198.2, 68.5)
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Connections:
- J1 pad TN: GND -> (no net)
Routing:
- net -12V: track 106.6 -> 88.1 mm
- net +12V: track 101.4 -> 96.7 mm
Other:
- board size 50 x 200 mm -> 46 x 172.1 mm
- board text added: "Rich Holmes / Feb 2023 CC0 1.0 https://github.com/holmesrichards/mults"
- board text removed: "Rich Holmes / August 2021 CC0 1.0 https://github.com/holmesrichards/mults"

Commit message: Pre fab tweaks
Parts:
- renumbered J2 to J1, J1 to J2
Routing:
- net Net-(U2C--): track 115.5 -> 116.8 mm
- net Net-(U1D--): track 141.0 -> 141.9 mm
