File: Hardware/Panel/multiples_panel/multiples_panel.kicad_pcb (KiCad board)
At the start: 2 copper layers, 50 x 200 mm, 15 parts

Commit message: gerbers
Parts:
- GRAF2: footprint ao_tht:CC0_logo -> AO_tht:CC0_logo
Other:
- net class Default removed
