File: Hardware/Panel/multiples_panel/multiples_panel.sch (KiCad schematic (older format))
At the start: 16 parts

Commit message: No NPTH specialization
Parts:
- removed GP1: Ground_point_for_NPTH, Kosmo_panel:Ground_point_for_NPTH, symbol Kosmo:Ground_point_for_NPTH
- H1, H10, H11, H12, H2, H4, H5, H7, H8, H9: footprint Kosmo_panel:Kosmo_Jack_Hole_NPTH -> Kosmo_panel:Kosmo_Jack_Hole
- H3, H6: footprint Kosmo_panel:Kosmo_Panel_Dual_Slotted_Mounting_Holes_NPTH -> Kosmo_panel:Kosmo_Panel_Dual_Slotted_Mounting_Holes
Changed lines of the file:
@@
 F 0 "H1" H 2135 1992 50  0000 L CNN
 F 1 "Jack_Hole" H 2135 1901 50  0000 L CNN
-F 2 "Kosmo_panel:Kosmo_Jack_Hole_NPTH" H 2000 2150 50  0001 C CNN
+F 2 "Kosmo_panel:Kosmo_Jack_Hole" H 2000 2150 50  0001 C CNN
 F 3 "" H 2000 2000 50  0001 C CNN
 	1    2000 2000
@@
 F 0 "H4" H 3135 1992 50  0000 L CNN
 F 1 "Jack_Hole" H 3135 1901 50  0000 L CNN
-F 2 "Kosmo_panel:Kosmo_Jack_Hole_NPTH" H 3000 2150 50  0001 C CNN
+F 2 "Kosmo_panel:Kosmo_Jack_Hole" H 3000 2150 50  0001 C CNN
 F 3 "" H 3000 2000 50  0001 C CNN
 	1    3000 2000
@@
 F 0 "H7" H 4135 1992 50  0000 L CNN
 F 1 "Jack_Hole" H 4135 1901 50  0000 L CNN
-F 2 "Kosmo_panel:Kosmo_Jack_Hole_NPTH" H 4000 2150 50  0001 C CNN
+F 2 "Kosmo_panel:Kosmo_Jack_Hole" H 4000 2150 50  0001 C CNN
 F 3 "" H 4000 2000 50  0001 C CNN
 	1    4000 2000
@@
 F 0 "H9" H 5135 1992 50  0000 L CNN
 F 1 "Jack_Hole" H 5135 1901 50  0000 L CNN
-F 2 "Kosmo_panel:Kosmo_Jack_Hole_NPTH" H 5000 2150 50  0001 C CNN
+F 2 "Kosmo_panel:Kosmo_Jack_Hole" H 5000 2150 50  0001 C CNN
 F 3 "" H 5000 2000 50  0001 C CNN
 	1    5000 2000
@@
 F 0 "H11" H 6135 1992 50  0000 L CNN
 F 1 "Jack_Hole" H 6135 1901 50  0000 L CNN
-F 2 "Kosmo_panel:Kosmo_Jack_Hole_NPTH" H 6000 2150 50  0001 C CNN
+F 2 "Kosmo_panel:Kosmo_Jack_Hole" H 6000 2150 50  0001 C CNN
 F 3 "" H 6000 2000 50  0001 C CNN
 	1    6000 2000
@@
 F 0 "H2" H 2135 2492 50  0000 L CNN
 F 1 "Jack_Hole" H 2135 2401 50  0000 L CNN
-F 2 "Kosmo_panel:Kosmo_Jack_Hole_NPTH" H 2000 2650 50  0001 C CNN
+F 2 "Kosmo_panel:Kosmo_Jack_Hole" H 2000 2650 50  0001 C CNN
 F 3 "" H 2000 2500 50  0001 C CNN
 	1    2000 2500
@@
 F 0 "H5" H 3135 2492 50  0000 L CNN
 F 1 "Jack_Hole" H 3135 2401 50  0000 L CNN
-F 2 "Kosmo_panel:Kosmo_Jack_Hole_NPTH" H 3000 2650 50  0001 C CNN
+F 2 "Kosmo_panel:Kosmo_Jack_Hole" H 3000 2650 50  0001 C CNN
 F 3 "" H 3000 2500 50  0001 C CNN
 	1    3000 2500
@@
 F 0 "H8" H 4135 2492 50  0000 L CNN
 F 1 "Jack_Hole" H 4135 2401 50  0000 L CNN
-F 2 "Kosmo_panel:Kosmo_Jack_Hole_NPTH" H 4000 2650 50  0001 C CNN
+F 2 "Kosmo_panel:Kosmo_Jack_Hole" H 4000 2650 50  0001 C CNN
 F 3 "" H 4000 2500 50  0001 C CNN
 	1    4000 2500
@@
 F 0 "H10" H 5135 2492 50  0000 L CNN
 F 1 "Jack_Hole" H 5135 2401 50  0000 L CNN
-F 2 "Kosmo_panel:Kosmo_Jack_Hole_NPTH" H 5000 2650 50  0001 C CNN
+F 2 "Kosmo_panel:Kosmo_Jack_Hole" H 5000 2650 50  0001 C CNN
 F 3 "" H 5000 2500 50  0001 C CNN
 	1    5000 2500
@@
 F 0 "H12" H 6135 2492 50  0000 L CNN
 F 1 "Jack_Hole" H 6135 2401 50  0000 L CNN
-F 2 "Kosmo_panel:Kosmo_Jack_Hole_NPTH" H 6000 2650 50  0001 C CNN
+F 2 "Kosmo_panel:Kosmo_Jack_Hole" H 6000 2650 50  0001 C CNN
 F 3 "" H 6000 2500 50  0001 C CNN
 	1    6000 2500
@@
 F 0 "H3" H 2100 3499 50  0000 L CNN
 F 1 "Mounting_Holes_Slotted" H 2100 3408 50  0000 L CNN
-F 2 "Kosmo_panel:Kosmo_Panel_Dual_Slotted_Mounting_Holes_NPTH" H 2000 3500 50  0001 C CNN
+F 2 "Kosmo_panel:Kosmo_Panel_Dual_Slotted_Mounting_Holes" H 2000 3500 50  0001 C CNN
 F 3 "" H 2000 3500 50  0001 C CNN
 	1    2000 3500
@@
 F 0 "H6" H 3600 3499 50  0000 L CNN
 F 1 "Mounting_Holes_Slotted" H 3600 3408 50  0000 L CNN
-F 2 "Kosmo_panel:Kosmo_Panel_Dual_Slotted_Mounting_Holes_NPTH" H 3500 3500 50  0001 C CNN
+F 2 "Kosmo_panel:Kosmo_Panel_Dual_Slotted_Mounting_Holes" H 3500 3500 50  0001 C CNN
 F 3 "" H 3500 3500 50  0001 C CNN
 	1    3500 3500
-	1    0    0    -1
-$EndComp
-$Comp
-L Kosmo:Ground_point_for_NPTH GP1
-U 1 1 611F52AB
-P 7200 2200
-F 0 "GP1" H 7280 2242 50  0000 L CNN
-F 1 "Ground_point_for_NPTH" H 7280 2151 50  0000 L CNN
-F 2 "Kosmo_panel:Ground_point_for_NPTH" H 7200 2200 50  0001 C CNN
-F 3 "~" H 7200 2200 50  0001 C CNN
-	1    7200 2200
 	1    0    0    -1
 $EndComp
@@
 Wire Wire Line
 	7000 2700 6000 2700
-Connection ~ 7000 2200
 Connection ~ 3000 2200
 Wire Wire Line

Commit message: gerbers
Parts:
- GRAF1, GRAF3: symbol ao_symbols:Graphic -> AO_symbols:Graphic
- GRAF2: footprint ao_tht:CC0_logo -> AO_tht:CC0_logo; symbol ao_symbols:Graphic -> AO_symbols:Graphic
Changed lines of the file:
@@
 	3150 3850 3500 3850
 $Comp
-L ao_symbols:Graphic GRAF1
+L AO_symbols:Graphic GRAF1
 U 1 1 611F7EE9
 P 2000 4600
@@
 $EndComp
 $Comp
-L ao_symbols:Graphic GRAF2
+L AO_symbols:Graphic GRAF2
 U 1 1 611F8831
 P 2000 4950
 F 0 "GRAF2" H 2278 4996 50  0000 L CNN
 F 1 "CC0 logo" H 2278 4905 50  0000 L CNN
-F 2 "ao_tht:CC0_logo" H 2000 4950 50  0001 C CNN
+F 2 "AO_tht:CC0_logo" H 2000 4950 50  0001 C CNN
 F 3 "" H 2000 4950 50  0001 C CNN
 F 4 "DNF" H 2000 4950 50  0001 C CNN "Config"
@@
 $EndComp
 $Comp
-L ao_symbols:Graphic GRAF3
+L AO_symbols:Graphic GRAF3
 U 1 1 611FC79C
 P 3000 4600
