File: Hardware/multiples/multiples.kicad_sch (KiCad schematic)
At the start: 39 parts, among them J1 Synth_power_2x5, J10 AudioJack2, J11 AudioJack2, J12 DIP-14, J13 DIP-14, J2 AudioJack2, J3 AudioJack2, J4 AudioJack2, J5 AudioJack2, J6 AudioJack2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

Commit message: Docs
Parts:
- GRAF1, GRAF2, GRAF3, TP1, TP2, TP3: now left out of the parts list
- J12, J13: SKU (none) -> A-004; Vendor (none) -> Tayda
Changed lines of the file:
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@@
   )
   (symbol (lib_id "AO_symbols:Graphic") (at 171.45 154.94 0) (unit 1)
-    (in_bom yes) (on_board yes) (dnp no)
+    (in_bom no) (on_board yes) (dnp no)
     (property "Reference" "GRAF1" (at 178.5112 153.7716 0)
       (effects (font (size 1.27 1.27)) (justify left))
@@
   )
   (symbol (lib_id "AO_symbols:Graphic") (at 196.85 154.94 0) (unit 1)
-    (in_bom yes) (on_board yes) (dnp no)
+    (in_bom no) (on_board yes) (dnp no)
     (property "Reference" "GRAF2" (at 203.9112 153.7716 0)
       (effects (font (size 1.27 1.27)) (justify left))
@@
   )
   (symbol (lib_id "AO_symbols:Graphic") (at 222.25 154.94 0) (unit 1)
-    (in_bom yes) (on_board yes) (dnp no)
+    (in_bom no) (on_board yes) (dnp no)
     (property "Reference" "GRAF3" (at 229.3112 153.7716 0)
       (effects (font (size 1.27 1.27)) (justify left))
@@
   )
   (symbol (lib_id "AO_symbols:TestPoint") (at 86.36 199.39 0) (unit 1)
-    (in_bom yes) (on_board yes) (dnp no) (fields_autoplaced)
+    (in_bom no) (on_board yes) (dnp no) (fields_autoplaced)
     (property "Reference" "TP2" (at 88.9 195.453 0)
       (effects (font (size 1.27 1.27)) (justify left))
@@
   )
   (symbol (lib_id "AO_symbols:TestPoint") (at 66.04 199.39 0) (unit 1)
-    (in_bom yes) (on_board yes) (dnp no) (fields_autoplaced)
+    (in_bom no) (on_board yes) (dnp no) (fields_autoplaced)
     (property "Reference" "TP1" (at 67.437 195.1795 0)
       (effects (font (size 1.27 1.27)) (justify left))
@@
   )
   (symbol (lib_id "AO_symbols:DIP-14") (at 110.49 151.13 0) (unit 1)
-    (in_bom yes) (on_board yes) (dnp no) (fields_autoplaced)
+    (in_bom yes) (on_board no) (dnp no) (fields_autoplaced)
     (property "Reference" "J12" (at 110.49 150.114 0)
       (effects (font (size 1.27 1.27)) hide)
@@
     )
     (property "Description" "" (at 110.49 151.13 0)
+      (effects (font (size 1.27 1.27)) hide)
+    )
+    (property "SKU" "A-004" (at 110.49 151.13 0)
+      (effects (font (size 1.27 1.27)) hide)
+    )
+    (property "Vendor" "Tayda" (at 110.49 151.13 0)
       (effects (font (size 1.27 1.27)) hide)
     )
@@
   )
   (symbol (lib_id "AO_symbols:DIP-14") (at 115.57 151.13 0) (unit 1)
-    (in_bom yes) (on_board yes) (dnp no) (fields_autoplaced)
+    (in_bom yes) (on_board no) (dnp no) (fields_autoplaced)
     (property "Reference" "J13" (at 115.57 150.114 0)
       (effects (font (size 1.27 1.27)) hide)
@@
       (effects (font (size 1.27 1.27)) hide)
     )
+    (property "SKU" "A-004" (at 115.57 151.13 0)
+      (effects (font (size 1.27 1.27)) hide)
+    )
+    (property "Vendor" "Tayda" (at 115.57 151.13 0)
+      (effects (font (size 1.27 1.27)) hide)
+    )
     (instances
       (project "multiples"
@@
   )
   (symbol (lib_id "AO_symbols:TestPoint") (at 107.95 199.39 0) (unit 1)
-    (in_bom yes) (on_board yes) (dnp no) (fields_autoplaced)
+    (in_bom no) (on_board yes) (dnp no) (fields_autoplaced)
     (property "Reference" "TP3" (at 110.49 195.453 0)
       (effects (font (size 1.27 1.27)) (justify left))
